Commit message: Add traditional Nav2 pipeline, mode arbitration, and odometry fusion
Responds to three pieces of feedback:

1. yolo_detector no longer drives the robot directly. It previously
   computed proportional steering from bounding-box position and
   published straight to cmd_vel, bypassing all obstacle/path
   reasoning. It now publishes vision_msgs/Detection2DArray; a new
   jetbot_nav package projects detections onto the ground plane
   (ground-plane-assumption / inverse perspective mapping, via the
   camera's known TF pose - added a proper camera_optical_frame to the
   URDF for this) into costmap obstacle points, and Nav2's standard
   controller/planner stack (no map_server/amcl - jetbot_slam is
   monocular-only, no occupancy grid yet) turns those into cmd_vel_nav.
   Deliberately camera-only for now; LiDAR integration is separate
   future work.

2. Removed Kyogin (a specific local machine name) from README.md and
   brain_research_report.md - genericized to "GPU server"/"GPU
   workstation" so the docs aren't tied to one person's hardware.

3. twist_mux doesn't blend commands, it's a priority selector, and its
   "lock" mechanism can't cleanly express "exactly one of two peer
   autonomous sources is live" (a lock blocks everything at or below a
   priority level, not a specific channel). Added jetbot_nav's
   mode_arbiter node upstream of twist_mux instead: it selects between
   the traditional planner and the VLA and republishes only that one to
   twist_mux's (renamed) autonomous input, so the joystick still always
   preempts whichever mode is active.

Also wires robot_localization's EKF to fuse motor_driver's open-loop
odometry into /odometry/filtered, taking over the odom->base_footprint
TF from motor_driver (new publish_tf param) - jetbot_slam's RTAB-Map is
unaffected, since it already reads that TF rather than owning it.

Two real bugs found and fixed by actually launching the new pipeline
rather than trusting the config on paper: ground_plane_projector's
origin was silently zeroed by a do_transform_vector3() call that
mutates its input in place (a Python reference-vs-copy bug caught by
comparing against a standalone hand-calculation, not by any error
message), and two Nav2 plugins needed pluginlib's package/ClassName
lookup form instead of the C++-namespace form several other Nav2
plugins accept. Verified end-to-end: obstacle projects to the correct
ground point, Nav2's costmap marks it, mode_arbiter forwards only the
selected pipeline, and the joystick still overrides either one.

Co-Authored-By: Claude Sonnet 5 <noreply@anthropic.com>

File: ros_ws/src/jetbot_description/urdf/jetbot.urdf (robot description, URDF)
Before this commit: robot jetbot, 5 links, 4 joints
Links:
- added link camera_optical_frame
Joints:
- added joint camera_optical_joint: type fixed, parent camera_link, child camera_optical_frame, origin xyz=0 0 0 rpy=-1.5707963267948966 0 -1.5707963267948966
